File: kicad/_autosave-const_curr_measure.kicad_pcb (KiCad board)
At the start: 4 copper layers, 160 x 100 mm, 102 parts, among them IC1 XTR110AG, J1 Conn_02x02_Counter_Clockwise, J10 1-726386-2, J11 1-726386-2, J12 09061152911, J13 Conn_01x05, J2 1-726386-2, J3 Conn_01x12, J4 1-726386-2, J5 Conn_01x03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

Commit message: * addded Ibom * added normal bom
Parts:
- TP1: value DAC_SHDN -> 1018.68
- TP10: value DAC_OUT -> 1018.68
- TP11: value SENSE+VDIV -> 1018.68
- TP12: value VREF_O -> 1018.68
- TP13: value VREF_ADJ -> 1018.68
- TP14: value ARD_A0 -> 1018.68
- TP15: value GND -> 1018.68
- TP16: value 5V -> 1018.68
- TP17: value DAC_OUT_FULL_SWING -> 1018.68
- TP18: value 20_EN -> 1018.68
- TP19: value 100_EN -> 1018.68
- TP2: value EN_ADD_03 -> 1018.68
- TP20: value 1000_EN -> 1018.68
- TP21: value 10000_EN -> 1018.68
- TP22: value 20_EN_Rel -> 1018.68
- TP23: value 100_EN_Rel -> 1018.68
- TP24: value 1000_EN_Rel -> 1018.68
- TP25: value 10000_EN_Rel -> 1018.68
- TP26: value TMP_S_OW -> 1018.68
- TP27: value 20mA_SHN -> 1018.68
- TP28: value 100mA_SHN -> 1018.68
- TP29: value 1000mA_SHN -> 1018.68
- TP3: value SPI_CS -> 1018.68
- TP30: value 10000mA_SHN -> 1018.68
- TP31: value EN_ADD_01 -> 1018.68
- TP32: value EN_ADD_02 -> 1018.68
- TP33: value ROT_POT_A -> 1018.68
- TP34: value ROT_POT_B -> 1018.68
- TP35: value Range_Down -> 1018.68
- TP36: value Range_up -> 1018.68
- TP37: value Rot_Enc_Button -> 1018.68
- TP38: value 5V ref -> 1018.68
- TP4: value SPI_SCK -> 1018.68
- TP5: value SPI_MOSI -> 1018.68
- TP6: value SENSE-VDIV -> 1018.68
- TP7: value SPAN_ADJ -> 1018.68
- TP8: value SRC_RES -> 1018.68
- TP9: value ARD_A1 -> 1018.68
