File: kicad/const_curr_measure.sch (KiCad schematic (older format))
At the start: 101 parts, among them IC1 XTR110AG, J1 Conn_02x02_Counter_Clockwise, J10 1-726386-2, J11 1-726386-2, J12 09061152911, J13 Conn_01x04, J2 1-726386-2, J3 Conn_01x06, J4 1-726386-2, J5 Conn_01x03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

Commit message: * most pcb routing
Parts:
- added TP38: 5V ref, TestPoint:TestPoint_THTPad_D2.5mm_Drill1.2mm, symbol Connector:TestPoint_Probe
- RV1: renamed from RV?; footprint (none) -> Potentiometer_THT:Potentiometer_Piher_PT-6-V_Vertical
- U3: renamed from U?; footprint Package_DIP:DIP-8_W7.62mm -> Package_DIP:DIP-8_W7.62mm_LongPads
- U4: renamed from U?; footprint (none) -> Package_DIP:DIP-8_W7.62mm_LongPads
- gave numbers to parts that had none: 2
Connections:
- wire segments 415 -> 417
Changed lines of the file:
@@
 	12150 2350 12000 2350
 $Comp
-L Analog_ADC:MCP3202 U?
+L Analog_ADC:MCP3202 U4
 U 1 1 6172EE79
 P 4200 3850
-F 0 "U?" H 4300 4531 50  0000 C CNN
+F 0 "U4" H 4300 4531 50  0000 C CNN
 F 1 "MCP3202" H 4300 4440 50  0000 C CNN
-F 2 "" H 4200 3750 50  0001 C CNN
+F 2 "Package_DIP:DIP-8_W7.62mm_LongPads" H 4200 3750 50  0001 C CNN
 F 3 "http://ww1.microchip.com/downloads/en/DeviceDoc/21034D.pdf" H 4200 4050 50  0001 C CNN
 	1    4200 3850
@@
 $EndComp
 $Comp
-L Reference_Voltage:REF02CP U?
+L Reference_Voltage:REF02CP U3
 U 1 1 60E60ABB
 P 1800 3900
-F 0 "U?" H 1850 4381 50  0000 C CNN
+F 0 "U3" H 1850 4381 50  0000 C CNN
 F 1 "REF02CP" H 1850 4290 50  0000 C CNN
-F 2 "Package_DIP:DIP-8_W7.62mm" H 2400 3650 50  0001 C CIN
+F 2 "Package_DIP:DIP-8_W7.62mm_LongPads" H 2400 3650 50  0001 C CIN
 F 3 "https://www.analog.com/media/en/technical-documentation/data-sheets/REF01_02_03.pdf" H 1850 3900 50  0001 C CIN
 	1    1800 3900
@@
 $EndComp
 $Comp
-L power:GND #PWR?
+L power:GND #PWR0150
 U 1 1 60F7C6ED
 P 4200 4450
-F 0 "#PWR?" H 4200 4200 50  0001 C CNN
+F 0 "#PWR0150" H 4200 4200 50  0001 C CNN
 F 1 "GND" H 4205 4277 50  0000 C CNN
 F 2 "" H 4200 4450 50  0001 C CNN
@@
 $EndComp
 $Comp
-L power:GND #PWR?
+L power:GND #PWR0151
 U 1 1 60FF7AB3
 P 1800 4300
-F 0 "#PWR?" H 1800 4050 50  0001 C CNN
+F 0 "#PWR0151" H 1800 4050 50  0001 C CNN
 F 1 "GND" H 1805 4127 50  0000 C CNN
 F 2 "" H 1800 4300 50  0001 C CNN
@@
 $EndComp
 $Comp
-L power:+5F #PWR?
+L power:+5F #PWR0159
 U 1 1 61023C01
 P 2500 3750
-F 0 "#PWR?" H 2500 3600 50  0001 C CNN
+F 0 "#PWR0159" H 2500 3600 50  0001 C CNN
 F 1 "+5F" H 2515 3923 50  0000 C CNN
 F 2 "" H 2500 3750 50  0001 C CNN
@@
 $EndComp
 $Comp
-L Device:R_POT RV?
+L Device:R_POT RV1
 U 1 1 610277AC
 P 2500 4000
-F 0 "RV?" H 2430 3954 50  0000 R CNN
+F 0 "RV1" H 2430 3954 50  0000 R CNN
 F 1 "10k" H 2430 4045 50  0000 R CNN
-F 2 "" H 2500 4000 50  0001 C CNN
+F 2 "Potentiometer_THT:Potentiometer_Piher_PT-6-V_Vertical" H 2500 4000 50  0001 C CNN
 F 3 "~" H 2500 4000 50  0001 C CNN
 	1    2500 4000
@@
 Connection ~ 2500 3800
 $Comp
-L power:+12V #PWR?
+L power:+12V #PWR0160
 U 1 1 6112B522
 P 1800 3450
-F 0 "#PWR?" H 1800 3300 50  0001 C CNN
+F 0 "#PWR0160" H 1800 3300 50  0001 C CNN
 F 1 "+12V" H 1815 3623 50  0000 C CNN
 F 2 "" H 1800 3450 50  0001 C CNN
@@
 	1800 3450 1800 3600
 $Comp
-L power:+5F #PWR?
+L power:+5F #PWR0161
 U 1 1 61159202
 P 4200 3300
-F 0 "#PWR?" H 4200 3150 50  0001 C CNN
+F 0 "#PWR0161" H 4200 3150 50  0001 C CNN
 F 1 "+5F" H 4215 3473 50  0000 C CNN
 F 2 "" H 4200 3300 50  0001 C CNN
@@
 ADC_CS
 $Comp
-L Device:C C?
+L Device:C C8
 U 1 1 613CF7D5
 P 5900 3900
-F 0 "C?" H 6015 3946 50  0000 L CNN
+F 0 "C8" H 6015 3946 50  0000 L CNN
 F 1 "100nF" H 6015 3855 50  0000 L CNN
 F 2 "Capacitor_THT:C_Rect_L7.2mm_W3.0mm_P5.00mm_FKS2_FKP2_MKS2_MKP2" H 5938 3750 50  0001 C CNN
@@
 $EndComp
 $Comp
-L power:GND #PWR?
+L power:GND #PWR0162
 U 1 1 613CF7DF
 P 5900 4150
-F 0 "#PWR?" H 5900 3900 50  0001 C CNN
+F 0 "#PWR0162" H 5900 3900 50  0001 C CNN
 F 1 "GND" H 5905 3977 50  0000 C CNN
 F 2 "" H 5900 4150 50  0001 C CNN
@@
 	1    0    0    -1
 $EndComp
-$Comp
-L power:+5V #PWR?
-U 1 1 613CF7E5
-P 5900 3600
-F 0 "#PWR?" H 5900 3450 50  0001 C CNN
-F 1 "+5V" H 5915 3773 50  0000 C CNN
-F 2 "" H 5900 3600 50  0001 C CNN
-F 3 "" H 5900 3600 50  0001 C CNN
-	1    5900 3600
-	1    0    0    -1
-$EndComp
 Wire Wire Line
 	5900 3600 5900 3750
@@
 	5900 4050 5900 4150
 $Comp
-L Device:C C?
+L Device:C C10
 U 1 1 6142A09B
 P 6500 3900
-F 0 "C?" H 6615 3946 50  0000 L CNN
+F 0 "C10" H 6615 3946 50  0000 L CNN
 F 1 "100nF" H 6615 3855 50  0000 L CNN
 F 2 "Capacitor_THT:C_Rect_L7.2mm_W3.0mm_P5.00mm_FKS2_FKP2_MKS2_MKP2" H 6538 3750 50  0001 C CNN
@@
 $EndComp
 $Comp
-L power:GND #PWR?
+L power:GND #PWR0164
 U 1 1 6142A0A1
 P 6500 4150
-F 0 "#PWR?" H 6500 3900 50  0001 C CNN
+F 0 "#PWR0164" H 6500 3900 50  0001 C CNN
 F 1 "GND" H 6505 3977 50  0000 C CNN
 F 2 "" H 6500 4150 50  0001 C CNN
@@
 	6500 4050 6500 4150
 $Comp
-L power:+5F #PWR?
+L power:+5F #PWR0165
 U 1 1 614577C2
 P 6500 3600
-F 0 "#PWR?" H 6500 3450 50  0001 C CNN
+F 0 "#PWR0165" H 6500 3450 50  0001 C CNN
 F 1 "+5F" H 6515 3773 50  0000 C CNN
 F 2 "" H 6500 3600 50  0001 C CNN
@@
 Text Notes 500  3200 0    100  ~ 0
 ADC-Section
+$Comp
+L power:+12V #PWR0163
+U 1 1 60EAAAC9
+P 5900 3600
+F 0 "#PWR0163" H 5900 3450 50  0001 C CNN
+F 1 "+12V" H 5915 3773 50  0000 C CNN
+F 2 "" H 5900 3600 50  0001 C CNN
+F 3 "" H 5900 3600 50  0001 C CNN
+	1    5900 3600
+	1    0    0    -1
+$EndComp
+$Comp
+L Connector:TestPoint_Probe TP38
+U 1 1 60F46120
+P 3050 3700
+F 0 "TP38" H 3007 3708 50  0000 R CNN
+F 1 "5V ref" H 3007 3799 50  0000 R CNN
+F 2 "TestPoint:TestPoint_THTPad_D2.5mm_Drill1.2mm" H 3250 3700 50  0001 C CNN
+F 3 "~" H 3250 3700 50  0001 C CNN
+	1    3050 3700
+	1    0    0    -1
+$EndComp
+Wire Wire Line
+	3050 3700 3050 3800
+Wire Wire Line
+	3050 3800 2500 3800
 $EndSCHEMATC

Commit message: * nearly finished pcb, changed front pcb connector to one big * added output enable switch net
Parts:
- removed J13: Conn_01x04, Connector_PinHeader_2.54mm:PinHeader_1x04_P2.54mm_Vertical, symbol Connector_Generic:Conn_01x04
- removed J3: Conn_01x06, Connector_PinHeader_2.54mm:PinHeader_1x06_P2.54mm_Vertical, symbol Connector_Generic:Conn_01x06
- added J3: Conn_01x12, Connector_PinHeader_2.54mm:PinHeader_1x12_P2.54mm_Vertical, symbol Connector_Generic:Conn_01x12
Connections:
- net labels added: OUTPUT_ENABLE
- net labels removed: ARDUINO_A0, ARDUINO_A1
- wire segments 417 -> 419
Other:
- note removed: "Front Power Connector\n"
- moved on the sheet: TP33, TP34, TP35, TP36, TP37
Changed lines of the file:
@@
 	1    0    0    -1
 $EndComp
-Text Notes 14300 3950 0    50   ~ 0
-Front Power Connector\n
 $Comp
 L power:GND #PWR0130
@@
 Text GLabel 15200 4850 0    50   Input ~ 0
 TEMP_SENS_OW
-Text GLabel 12850 800  2    50   Input ~ 0
-ARDUINO_A0
-Text GLabel 12850 900  2    50   Input ~ 0
-ARDUINO_A1
 $Comp
 L power:+5V #PWR0134
@@
 L power:GND #PWR0138
 U 1 1 62009784
-P 14150 2950
-F 0 "#PWR0138" H 14150 2700 50  0001 C CNN
-F 1 "GND" H 14155 2777 50  0000 C CNN
-F 2 "" H 14150 2950 50  0001 C CNN
-F 3 "" H 14150 2950 50  0001 C CNN
-	1    14150 2950
-	1    0    0    -1
-$EndComp
-$Comp
-L Connector_Generic:Conn_01x06 J3
-U 1 1 62082BB7
-P 15300 2650
-F 0 "J3" H 15380 2642 50  0000 L CNN
-F 1 "Conn_01x06" H 15380 2551 50  0000 L CNN
-F 2 "Connector_PinHeader_2.54mm:PinHeader_1x06_P2.54mm_Vertical" H 15300 2650 50  0001 C CNN
-F 3 "~" H 15300 2650 50  0001 C CNN
-	1    15300 2650
+P 13300 2250
+F 0 "#PWR0138" H 13300 2000 50  0001 C CNN
+F 1 "GND" H 13305 2077 50  0000 C CNN
+F 2 "" H 13300 2250 50  0001 C CNN
+F 3 "" H 13300 2250 50  0001 C CNN
+	1    13300 2250
 	1    0    0    -1
 $EndComp
@@
 L Connector:TestPoint_Probe TP34
 U 1 1 6214B38F
-P 14850 3250
-F 0 "TP34" H 15003 3351 50  0000 L CNN
-F 1 "ROT_POT_B" H 15003 3260 50  0000 L CNN
-F 2 "TestPoint:TestPoint_THTPad_D2.5mm_Drill1.2mm" H 15050 3250 50  0001 C CNN
-F 3 "~" H 15050 3250 50  0001 C CNN
-	1    14850 3250
+P 14550 2550
+F 0 "TP34" H 14703 2651 50  0000 L CNN
+F 1 "ROT_POT_B" H 14703 2560 50  0000 L CNN
+F 2 "TestPoint:TestPoint_THTPad_D2.5mm_Drill1.2mm" H 14750 2550 50  0001 C CNN
+F 3 "~" H 14750 2550 50  0001 C CNN
+	1    14550 2550
 	1    0    0    -1
 $EndComp
@@
 L Connector:TestPoint_Probe TP33
 U 1 1 62164151
-P 14750 3400
-F 0 "TP33" H 14902 3501 50  0000 L CNN
-F 1 "ROT_POT_A" H 14902 3410 50  0000 L CNN
-F 2 "TestPoint:TestPoint_THTPad_D2.5mm_Drill1.2mm" H 14950 3400 50  0001 C CNN
-F 3 "~" H 14950 3400 50  0001 C CNN
-	1    14750 3400
-	1    0    0    -1
-$EndComp
-Wire Wire Line
-	14850 3250 14850 2550
-Wire Wire Line
-	14850 2550 14450 2550
-Connection ~ 14850 2550
-Wire Wire Line
-	14450 2650 14750 2650
-Wire Wire Line
-	14750 3400 14750 2650
-Connection ~ 14750 2650
+P 14450 2700
+F 0 "TP33" H 14602 2801 50  0000 L CNN
+F 1 "ROT_POT_A" H 14602 2710 50  0000 L CNN
+F 2 "TestPoint:TestPoint_THTPad_D2.5mm_Drill1.2mm" H 14650 2700 50  0001 C CNN
+F 3 "~" H 14650 2700 50  0001 C CNN
+	1    14450 2700
+	1    0    0    -1
+$EndComp
+Wire Wire Line
+	14550 2550 14550 1850
+Wire Wire Line
+	14550 1850 14150 1850
+Connection ~ 14550 1850
+Wire Wire Line
+	14150 1950 14450 1950
+Wire Wire Line
+	14450 2700 14450 1950
+Connection ~ 14450 1950
 $Comp
 L Connector:TestPoint_Probe TP26
@@
 Wire Wire Line
 	10500 7600 10800 7600
-Text Notes 14300 2350 0    50   ~ 0
+Text Notes 14000 1650 0    50   ~ 0
 Front I/O Connector\n
 Wire Wire Line
@@
 Text GLabel 8150 1550 0    50   Input ~ 0
 FET_SOURCE
-Text GLabel 14450 2550 0    50   Input ~ 0
+Text GLabel 14150 1850 0    50   Input ~ 0
 ROT_POT_B
-Text GLabel 14450 2650 0    50   Input ~ 0
+Text GLabel 14150 1950 0    50   Input ~ 0
 ROT_POT_A
 Wire Wire Line
@@
 $EndComp
 Wire Wire Line
-	14450 2750 14650 2750
-$Comp
-L Connector_Generic:Conn_01x04 J13
-U 1 1 615CE8E4
-P 15000 1450
-F 0 "J13" H 15080 1442 50  0000 L CNN
-F 1 "Conn_01x04" H 15080 1351 50  0000 L CNN
-F 2 "Connector_PinHeader_2.54mm:PinHeader_1x04_P2.54mm_Vertical" H 15000 1450 50  0001 C CNN
-F 3 "~" H 15000 1450 50  0001 C CNN
-	1    15000 1450
-	1    0    0    -1
-$EndComp
+	14150 2050 14350 2050
 $Comp
 L power:GND #PWR0131
@@
 Text GLabel 5750 1350 2    50   Input ~ 0
 10000mA_Shunt_Sense_-
-Text GLabel 14450 2750 0    50   Input ~ 0
+Text GLabel 14150 2050 0    50   Input ~ 0
 RANGE_UP
-Text GLabel 14450 2850 0    50   Input ~ 0
+Text GLabel 14150 2150 0    50   Input ~ 0
 RANGE_DOWN
 $Comp
 L Connector:TestPoint_Probe TP36
 U 1 1 619CC181
-P 14650 3550
-F 0 "TP36" H 14803 3651 50  0000 L CNN
-F 1 "Range_up" H 14803 3560 50  0000 L CNN
-F 2 "TestPoint:TestPoint_THTPad_D2.5mm_Drill1.2mm" H 14850 3550 50  0001 C CNN
-F 3 "~" H 14850 3550 50  0001 C CNN
-	1    14650 3550
+P 14350 2850
+F 0 "TP36" H 14503 2951 50  0000 L CNN
+F 1 "Range_up" H 14503 2860 50  0000 L CNN
+F 2 "TestPoint:TestPoint_THTPad_D2.5mm_Drill1.2mm" H 14550 2850 50  0001 C CNN
+F 3 "~" H 14550 2850 50  0001 C CNN
+	1    14350 2850
 	1    0    0    -1
 $EndComp
@@
 L Connector:TestPoint_Probe TP35
 U 1 1 619CC187
-P 14550 3700
-F 0 "TP35" H 14702 3801 50  0000 L CNN
-F 1 "Range_Down" H 14702 3710 50  0000 L CNN
-F 2 "TestPoint:TestPoint_THTPad_D2.5mm_Drill1.2mm" H 14750 3700 50  0001 C CNN
-F 3 "~" H 14750 3700 50  0001 C CNN
-	1    14550 3700
-	1    0    0    -1
-$EndComp
-Connection ~ 14650 2750
-Wire Wire Line
-	14450 2850 14550 2850
-Wire Wire Line
-	14650 2750 14650 3550
-Connection ~ 14550 2850
-Wire Wire Line
-	14550 2850 14550 3700
+P 14250 3000
+F 0 "TP35" H 14402 3101 50  0000 L CNN
+F 1 "Range_Down" H 14402 3010 50  0000 L CNN
+F 2 "TestPoint:TestPoint_THTPad_D2.5mm_Drill1.2mm" H 14450 3000 50  0001 C CNN
+F 3 "~" H 14450 3000 50  0001 C CNN
+	1    14250 3000
+	1    0    0    -1
+$EndComp
+Connection ~ 14350 2050
+Wire Wire Line
+	14150 2150 14250 2150
+Wire Wire Line
+	14350 2050 14350 2850
+Connection ~ 14250 2150
 $Comp
 L Connector:TestPoint_Probe TP37
 U 1 1 61A9CEDF
-P 14950 3100
-F 0 "TP37" H 15103 3201 50  0000 L CNN
-F 1 "Rot_Enc_Button" H 15103 3110 50  0000 L CNN
-F 2 "TestPoint:TestPoint_THTPad_D2.5mm_Drill1.2mm" H 15150 3100 50  0001 C CNN
-F 3 "~" H 15150 3100 50  0001 C CNN
-	1    14950 3100
-	1    0    0    -1
-$EndComp
-Wire Wire Line
-	14950 3100 14950 2450
-Wire Wire Line
-	14950 2450 15100 2450
-Wire Wire Line
-	14850 2550 15100 2550
-Wire Wire Line
-	14750 2650 15100 2650
-Wire Wire Line
-	14650 2750 15100 2750
-Wire Wire Line
-	14550 2850 15100 2850
-Wire Wire Line
-	14150 2950 15100 2950
-Text GLabel 14450 2450 0    50   Input ~ 0
+P 14650 2400
+F 0 "TP37" H 14803 2501 50  0000 L CNN
+F 1 "Rot_Enc_Button" H 14803 2410 50  0000 L CNN
+F 2 "TestPoint:TestPoint_THTPad_D2.5mm_Drill1.2mm" H 14850 2400 50  0001 C CNN
+F 3 "~" H 14850 2400 50  0001 C CNN
+	1    14650 2400
+	1    0    0    -1
+$EndComp
+Wire Wire Line
+	14650 2400 14650 1750
+Wire Wire Line
+	14650 1750 14800 1750
+Wire Wire Line
+	14550 1850 14800 1850
+Wire Wire Line
+	14450 1950 14800 1950
+Wire Wire Line
+	14350 2050 14800 2050
+Wire Wire Line
+	14250 2150 14800 2150
+Text GLabel 14150 1750 0    50   Input ~ 0
 Rot_Enc_But
 Wire Wire Line
-	14450 2450 14950 2450
-Connection ~ 14950 2450
+	14150 1750 14650 1750
+Connection ~ 14650 1750
 $Comp
 L Connector_Generic:Conn_01x03 J5
@@
 Wire Wire Line
 	12150 2750 12000 2750
-Wire Wire Line
-	12150 2450 12000 2450
-Wire Wire Line
-	12150 2350 12000 2350
 $Comp
 L Analog_ADC:MCP3202 U4
@@
 Wire Wire Line
 	3050 3800 2500 3800
+$Comp
+L power:GND #PWR0166
+U 1 1 60EAA45C
+P 14000 2500
+F 0 "#PWR0166" H 14000 2250 50  0001 C CNN
+F 1 "GND" H 14000 2350 50  0000 C CNN
+F 2 "" H 14000 2500 50  0000 C CNN
+F 3 "" H 14000 2500 50  0000 C CNN
+	1    14000 2500
+	1    0    0    -1
+$EndComp
+Wire Wire Line
+	14000 2500 14000 2450
+Text GLabel 12150 2350 2    50   Input ~ 0
+OUTPUT_ENABLE
+Wire Wire Line
+	12150 2350 12000 2350
+Text GLabel 14100 2350 0    50   Input ~ 0
+OUTPUT_ENABLE
+Wire Wire Line
+	14250 2150 14250 3000
+Wire Wire Line
+	14800 2250 13300 2250
+Wire Wire Line
+	14000 2450 14800 2450
+Wire Wire Line
+	14100 2350 14800 2350
+$Comp
+L Connector_Generic:Conn_01x12 J3
+U 1 1 611B7451
+P 15000 1850
+F 0 "J3" H 15080 1842 50  0000 L CNN
+F 1 "Conn_01x12" H 15080 1751 50  0000 L CNN
+F 2 "Connector_PinHeader_2.54mm:PinHeader_1x12_P2.54mm_Vertical" H 15000 1850 50  0001 C CNN
+F 3 "~" H 15000 1850 50  0001 C CNN
+	1    15000 1850
+	1    0    0    -1
+$EndComp
 $EndSCHEMATC

Commit message: * first revision will order this version
Parts:
- added J13: Conn_01x05, Connector_PinHeader_2.54mm:PinHeader_1x05_P2.54mm_Vertical, symbol Connector_Generic:Conn_01x05
Changed lines of the file:
@@
+	1    0    0    -1
+$EndComp
+$Comp
+L Connector_Generic:Conn_01x05 J13
+U 1 1 6130893A
+P 12600 4550
+F 0 "J13" H 12680 4592 50  0000 L CNN
+F 1 "Conn_01x05" H 12680 4501 50  0000 L CNN
+F 2 "Connector_PinHeader_2.54mm:PinHeader_1x05_P2.54mm_Vertical" H 12600 4550 50  0001 C CNN
+F 3 "~" H 12600 4550 50  0001 C CNN
+	1    12600 4550
 	1    0    0    -1
 $EndComp
